File: hardware/test_SGTL5000/codec.kicad_sch (KiCad schematic)
At the start: 5 parts

Commit message: schema
Parts:
- added J301: LINEIN_R, Connector_Coaxial:SMA_Amphenol_132134_Vertical, symbol Connector:Conn_Coaxial
- added J302: LINEIN_L, Connector_Coaxial:SMA_Amphenol_132134_Vertical, symbol Connector:Conn_Coaxial
- added J303: MIC, Connector_Coaxial:SMA_Amphenol_132134_Vertical, symbol Connector:Conn_Coaxial
- added J304: LINEOUT_L, Connector_Coaxial:SMA_Amphenol_132134_Vertical, symbol Connector:Conn_Coaxial
- added J305: LINEOUT_R, symbol Connector:Conn_Coaxial
- C301, C302, C303, C304: renamed from C?; footprint Capacitor_SMD:C_0603_1608Metric -> Capacitor_SMD:C_0402_1005Metric
- gave numbers to parts that had none: 1
Connections:
- net GND: now also J301.2 (Ext), J302.2 (Ext), J303.2 (Ext), J304.2 (Ext), J305.2 (Ext)
- net MIC: now reaches U301.10 (MIC)
- net MIC: now also J303.1 (In)
- net VAG: now reaches C301.1, U301.5 (VAG)
- net LINEOUT_R: now reaches U301.6 (LINEOUT_R)
- net LINEOUT_R: now also J305.1 (In)
- net LINEOUT_L: now reaches U301.7 (LINEOUT_L)
- net LINEOUT_L: now also J304.1 (In)
- net LINEIN_R: now reaches U301.8 (LINEIN_R)
- net LINEIN_R: now also J301.1 (In)
- net LINEIN_L: now reaches U301.9 (LINEIN_L)
- net LINEIN_L: now also J302.1 (In)
- no-connect marks 0 -> 4
Other:
- moved on the sheet: C301

Commit message: routing
Parts:
- J301, J302, J303, J304: footprint Connector_Coaxial:SMA_Amphenol_132134_Vertical -> WITNS:BNC_RS-PRO_546-4027
- J305: footprint (none) -> WITNS:BNC_RS-PRO_546-4027
