File: hardware/test_SGTL5000/power.kicad_sch (KiCad schematic)
At the start: 17 parts

Commit message: schema
Parts:
- added TP501, TP502, TP503: TestPoint, TestPoint:TestPoint_Pad_D1.5mm, symbol Connector:TestPoint
- gave numbers to parts that had none: 16
Connections:
- net +1V8: now also TP503.1
- net +3.3VA: now also TP501.1
- net +3V3: now also TP502.1
Other:
- moved on the sheet: C501, C502, C503, C504, C505, C506, D501, D502, D503, F501, FB1, R501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

Commit message: routing
Parts:
- C501, C502, C503, C504, C505, C506: footprint Capacitor_SMD:C_0603_1608Metric_Pad1.08x0.95mm_HandSolder -> Capacitor_SMD:C_0603_1608Metric
- D501, D502, D503: footprint LED_SMD:LED_0603_1608Metric_Pad1.05x0.95mm_HandSolder -> LED_SMD:LED_0603_1608Metric
- F501: footprint Fuse:Fuse_1206_3216Metric_Pad1.42x1.75mm_HandSolder -> Fuse:Fuse_1206_3216Metric
- R501, R502, R503: footprint Resistor_SMD:R_0603_1608Metric_Pad0.98x0.95mm_HandSolder -> Resistor_SMD:R_0603_1608Metric
