File: hardware/test_SGTL5000/test_SGTL5000.kicad_sch (KiCad schematic)
At the start: 0 parts

Commit message: schema
Parts:
- added H101, H102, H103, H104: MountingHole_Pad, MountingHole:MountingHole_3.2mm_M3_Pad_Via, symbol Mechanical:MountingHole_Pad
- added JP101, JP102, JP103, JP104, JP105, JP106, JP107: SolderJumper_2_Open, Resistor_SMD:R_0603_1608Metric, symbol Jumper:SolderJumper_2_Open
- added TP101, TP102, TP103, TP104, TP105, TP106, TP107: TestPoint, TestPoint:TestPoint_Pad_D1.5mm, symbol Connector:TestPoint
Connections:
- net CODEC/I2C_SCL: now also JP106.2 (B)
- net CODEC/I2C_SDA: now also JP107.2 (B)
- net CODEC/I2S_DIN: now also JP104.2 (B)
- net CODEC/I2S_DOUT: now also JP105.2 (B)
- net CODEC/I2S_LRCLK: now also JP103.2 (B)
- net CODEC/I2S_SCLK: now also JP102.2 (B)
- net CODEC/SYS_MCLK: now also JP101.2 (B)
- new net GND: H101.1, H102.1, H103.1, H104.1
- new net STM32/I2C_SCL: JP106.1 (A), TP106.1
- new net STM32/I2C_SDA: JP107.1 (A), TP107.1
- new net STM32/I2S_DIN: JP104.1 (A), TP104.1
- new net STM32/I2S_DOUT: JP105.1 (A), TP105.1
- new net STM32/I2S_LRCLK: JP103.1 (A), TP103.1
- new net STM32/I2S_SCLK: JP102.1 (A), TP102.1
- new net STM32/SYS_MCLK: JP101.1 (A), TP101.1
