File: hardware/test_SGTL5000/usb.kicad_sch (KiCad schematic)
At the start: 4 parts

Commit message: schema
Parts:
- gave numbers to parts that had none: 4
Changed lines of the file:
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@@
   (junction (at 127 96.52) (diameter 0) (color 0 0 0 0)
+  )
+  (junction (at 110.49 121.92) (diameter 0) (color 0 0 0 0)
   )
   (no_connect (at 102.87 120.65))
@@
     (stroke (width 0) (type default) (color 0 0 0 0))
   )
+  (wire (pts (xy 114.3 123.19) (xy 114.3 121.92))
+    (stroke (width 0) (type default) (color 0 0 0 0))
+  )
   (wire (pts (xy 127 96.52) (xy 127 97.79))
     (stroke (width 0) (type default) (color 0 0 0 0))
@@
     (stroke (width 0) (type default) (color 0 0 0 0))
   )
+  (wire (pts (xy 110.49 121.92) (xy 110.49 120.65))
+    (stroke (width 0) (type default) (color 0 0 0 0))
+  )
   (wire (pts (xy 127 96.52) (xy 163.83 96.52))
     (stroke (width 0) (type default) (color 0 0 0 0))
@@
     (stroke (width 0) (type default) (color 0 0 0 0))
   )
+  (wire (pts (xy 110.49 125.73) (xy 110.49 121.92))
+    (stroke (width 0) (type default) (color 0 0 0 0))
+  )
   (wire (pts (xy 176.53 98.425) (xy 176.53 97.79))
     (stroke (width 0) (type default) (color 0 0 0 0))
@@
     (stroke (width 0) (type default) (color 0 0 0 0))
   )
+  (wire (pts (xy 114.3 121.92) (xy 110.49 121.92))
+    (stroke (width 0) (type default) (color 0 0 0 0))
+  )
   (wire (pts (xy 125.73 100.33) (xy 127 100.33))
     (stroke (width 0) (type default) (color 0 0 0 0))
@@
   (wire (pts (xy 163.83 111.76) (xy 157.48 111.76))
     (stroke (width 0) (type default) (color 0 0 0 0))
-  )
-  (label "VBUS" (at 147.32 104.14 90)
-    (effects (font (size 1.27 1.27)) (justify left bottom))
   )
   (label "D-" (at 128.27 96.52 0)
@@
     (effects (font (size 1.27 1.27)) (justify right))
   )
-  (symbol (lib_id "power:GND") (at 110.49 120.65 0) (unit 1)
-    (in_bom yes) (on_board yes) (fields_autoplaced)
-    (property "Reference" "#PWR?" (id 0) (at 110.49 127 0)
-      (effects (font (size 1.27 1.27)) hide)
-    )
-    (property "Value" "GND" (id 1) (at 110.49 125.73 0))
-    (property "Footprint" "" (id 2) (at 110.49 120.65 0)
-      (effects (font (size 1.27 1.27)) hide)
-    )
-    (property "Datasheet" "" (id 3) (at 110.49 120.65 0)
+  (hierarchical_label "VBUS" (shape input) (at 147.32 104.14 90)
+    (effects (font (size 1.27 1.27)) (justify left))
+  )
+  (symbol (lib_id "power:GND") (at 110.49 125.73 0) (unit 1)
+    (in_bom yes) (on_board yes) (fields_autoplaced)
+    (property "Reference" "#PWR0401" (id 0) (at 110.49 132.08 0)
+      (effects (font (size 1.27 1.27)) hide)
+    )
+    (property "Value" "GND" (id 1) (at 110.49 130.81 0))
+    (property "Footprint" "" (id 2) (at 110.49 125.73 0)
+      (effects (font (size 1.27 1.27)) hide)
+    )
+    (property "Datasheet" "" (id 3) (at 110.49 125.73 0)
       (effects (font (size 1.27 1.27)) hide)
     )
@@
   (symbol (lib_id "Device:R_Small") (at 176.53 95.25 0) (unit 1)
     (in_bom yes) (on_board yes)
-    (property "Reference" "R?" (id 0) (at 177.8 93.98 0)
+    (property "Reference" "R402" (id 0) (at 177.8 93.98 0)
       (effects (font (size 1.27 1.27)) (justify left))
     )
@@
   (symbol (lib_id "Device:R_Small") (at 170.18 95.25 0) (unit 1)
     (in_bom yes) (on_board yes)
-    (property "Reference" "R?" (id 0) (at 171.45 93.98 0)
+    (property "Reference" "R401" (id 0) (at 171.45 93.98 0)
       (effects (font (size 1.27 1.27)) (justify left))
     )
@@
   (symbol (lib_id "Connector:USB_C_Receptacle_USB2.0") (at 110.49 97.79 0) (unit 1)
     (in_bom yes) (on_board yes) (fields_autoplaced)
-    (property "Reference" "J?" (id 0) (at 110.49 74.295 0))
+    (property "Reference" "J401" (id 0) (at 110.49 74.295 0))
     (property "Value" "USB_C_Receptacle_USB2.0" (id 1) (at 110.49 76.835 0))
     (property "Footprint" "Connector_USB:USB_C_Receptacle_HRO_TYPE-C-31-M-12" (id 2) (at 114.3 97.79 0)
@@
   (symbol (lib_id "Power_Protection:USBLC6-2SC6") (at 147.32 114.3 0) (unit 1)
     (in_bom yes) (on_board yes)
-    (property "Reference" "U?" (id 0) (at 148.59 102.87 0)
+    (property "Reference" "U401" (id 0) (at 148.59 102.87 0)
       (effects (font (size 1.27 1.27)) (justify left))
     )
@@
   (symbol (lib_id "power:GND") (at 170.18 99.695 0) (unit 1)
     (in_bom yes) (on_board yes)
-    (property "Reference" "#PWR?" (id 0) (at 170.18 106.045 0)
+    (property "Reference" "#PWR0403" (id 0) (at 170.18 106.045 0)
       (effects (font (size 1.27 1.27)) hide)
     )
@@
   (symbol (lib_id "power:GND") (at 147.32 124.46 0) (unit 1)
     (in_bom yes) (on_board yes) (fields_autoplaced)
-    (property "Reference" "#PWR?" (id 0) (at 147.32 130.81 0)
+    (property "Reference" "#PWR0402" (id 0) (at 147.32 130.81 0)
       (effects (font (size 1.27 1.27)) hide)
     )
@@
       (effects (font (size 1.27 1.27)) hide)
     )
+    (pin "1")
+  )
+  (symbol (lib_id "power:PWR_FLAG") (at 114.3 123.19 180) (unit 1)
+    (in_bom yes) (on_board yes) (fields_autoplaced)
+    (property "Reference" "#FLG0101" (id 0) (at 114.3 125.095 0)
+      (effects (font (size 1.27 1.27)) hide)
+    )
+    (property "Value" "PWR_FLAG" (id 1) (at 116.84 124.4599 0)
+      (effects (font (size 1.27 1.27)) (justify right))
+    )
+    (property "Footprint" "" (id 2) (at 114.3 123.19 0)
+      (effects (font (size 1.27 1.27)) hide)
+    )
+    (property "Datasheet" "~" (id 3) (at 114.3 123.19 0)
+      (effects (font (size 1.27 1.27)) hide)
+    )

Commit message: routing
Parts:
- R401, R402: footprint Resistor_SMD:R_0603_1608Metric_Pad0.98x0.95mm_HandSolder -> Resistor_SMD:R_0603_1608Metric
