File: hardware/test_SGTL5000/stm32.kicad_sch (KiCad schematic)
At the start: 18 parts

Commit message: schema
Parts:
- C201: renamed from C?; footprint Capacitor_SMD:C_0603_1608Metric -> Capacitor_SMD:C_0402_1005Metric
- C204, C208: renamed from C?; footprint Capacitor_SMD:C_0603_1608Metric_Pad1.08x0.95mm_HandSolder -> Capacitor_SMD:C_0603_1608Metric
- C205, C206, C207: renamed from C?; footprint Capacitor_SMD:C_0603_1608Metric_Pad1.08x0.95mm_HandSolder -> Capacitor_SMD:C_0402_1005Metric
- gave numbers to parts that had none: 12
Connections:
- net SWCLK: now also U201.24 (PA14)
- net SWDIO: now also U201.23 (PA13)
- net SWO: now also U201.26 (PB3)
- no-connect marks 11 -> 8

Commit message: Started routing
Parts:
- C202, C203: footprint Capacitor_SMD:C_0603_1608Metric -> Capacitor_SMD:C_0402_1005Metric
- R204: footprint Resistor_SMD:R_0603_1608Metric -> Resistor_SMD:R_0402_1005Metric
Changed lines of the file:
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@@
       (effects (font (size 1.27 1.27)))
     )
-    (property "Footprint" "Resistor_SMD:R_0603_1608Metric" (at 199.39 81.28 0)
+    (property "Footprint" "Resistor_SMD:R_0402_1005Metric" (at 199.39 81.28 0)
       (effects (font (size 1.27 1.27)) hide)
     )
@@
       (effects (font (size 1.27 1.27)))
     )
-    (property "Footprint" "Capacitor_SMD:C_0603_1608Metric" (at 179.07 96.52 0)
+    (property "Footprint" "Capacitor_SMD:C_0402_1005Metric" (at 179.07 96.52 0)
       (effects (font (size 1.27 1.27)) hide)
     )
@@
       (effects (font (size 1.27 1.27)))
     )
-    (property "Footprint" "Capacitor_SMD:C_0603_1608Metric" (at 179.07 86.36 0)
-      (effects (font (size 1.27 1.27)) hide)
-    )
+    (property "Footprint" "Capacitor_SMD:C_0402_1005Metric" (at 179.07 86.36 0)
+      (effects (font (size 1.27 1.27)) hide)
+    )

Commit message: routing
Connections:
- net LED1: now also U201.10 (PA5); no longer U201.5 (PA0)
- net LED2: now also U201.9 (PA4); no longer U201.6 (PA1)
Changed lines of the file:
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@@
   )
   (no_connect (at 209.55 111.76))
-  (no_connect (at 240.03 86.36))
+  (no_connect (at 240.03 78.74))
   (no_connect (at 240.03 91.44))
   (no_connect (at 209.55 96.52))
-  (no_connect (at 240.03 88.9))
   (no_connect (at 76.2 60.96))
+  (no_connect (at 240.03 76.2))
   (no_connect (at 240.03 93.98))
   (no_connect (at 76.2 55.88))
@@
     (effects (font (size 1.27 1.27)) (justify right bottom))
   )
-  (label "LED2" (at 240.03 78.74 0) (fields_autoplaced)
+  (label "LED2" (at 240.03 86.36 0) (fields_autoplaced)
     (effects (font (size 1.27 1.27)) (justify left bottom))
   )
@@
     (effects (font (size 1.27 1.27)) (justify left bottom))
   )
-  (label "LED1" (at 240.03 76.2 0) (fields_autoplaced)
-    (effects (font (size 1.27 1.27)) (justify left bottom))
-  )
+  (label "LED1" (at 240.03 88.9 0) (fields_autoplaced)
+    (effects (font (size 1.27 1.27)) (justify left bottom))
+  )
