File: hardware/test_SGTL5000/test_SGTL5000.kicad_pcb (KiCad board)
At the start: 2 copper layers, 68 x 68 mm, 70 parts, among them J201 SWD, J301 LINEIN_R, J302 LINEIN_L, J303 MIC, J304 LINEOUT_L, J305 LINEOUT_R, J401 USB_C_Receptacle_USB2.0, SW201 RST, U201 STM32G431KBT6, U301 SGTL5000XNLA3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

Commit message: routing
Parts:
- C501, C502, C503, C504, C505, C506: footprint Capacitor_SMD:C_0603_1608Metric_Pad1.08x0.95mm_HandSolder -> Capacitor_SMD:C_0603_1608Metric
- D501, D502, D503: footprint LED_SMD:LED_0603_1608Metric_Pad1.05x0.95mm_HandSolder -> LED_SMD:LED_0603_1608Metric
- F501: footprint Fuse:Fuse_1206_3216Metric_Pad1.42x1.75mm_HandSolder -> Fuse:Fuse_1206_3216Metric
- FB1: footprint Inductor_SMD:L_0805_2012Metric_Pad1.05x1.20mm_HandSolder -> Inductor_SMD:L_0805_2012Metric
- J301, J302, J303, J304, J305: footprint Connector_Coaxial:SMA_Amphenol_132134_Vertical -> WITNS:BNC_RS-PRO_546-4027
- R401, R402, R501, R502, R503: footprint Resistor_SMD:R_0603_1608Metric_Pad0.98x0.95mm_HandSolder -> Resistor_SMD:R_0603_1608Metric
- moved J302 31.4 mm to (30.5, 78.0)
- moved C502 19.9 mm to (71.0, 31.0), turned to 0 degrees
- moved J304 19.8 mm to (58.5, 78.0)
- moved U502 16.3 mm to (71.0, 28.0), turned to 90 degrees
- moved J301 13.4 mm to (42.0, 78.0)
- moved C505 13.0 mm to (71.0, 25.0), turned to 0 degrees
- moved D502 11.2 mm to (71.0, 23.0), turned to 180 degrees
- moved J303 10.8 mm to (30.5, 65.5)
- moved R502 9.85 mm to (71.0, 21.0), turned to 0 degrees
- moved C303 9.22 mm to (46.2, 67.6), turned to -90 degrees
- moved JP102 8.60 mm to (48.0, 58.0)
- moved F501 8.00 mm to (80.0, 31.0)
- moved FB1 8.00 mm to (77.0, 31.0)
- moved J401 8.00 mm to (80.0, 40.0)
- moved R401 8.00 mm to (72.0, 35.0)
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Routing:
- net /CODEC/MIC: track 0.00 -> 69.6 mm
- net /CODEC/LINEIN_L: track 0.00 -> 38.4 mm
- net /CODEC/LINEOUT_R: track 0.00 -> 26.7 mm, vias 0 -> 1
- net /CODEC/LINEIN_R: track 0.00 -> 23.7 mm
- net /STM32/I2S_LRCLK: track 0.00 -> 20.7 mm
- net /STM32/I2S_SCLK: track 0.00 -> 18.1 mm
- net /CODEC/I2C_SCL: track 0.00 -> 18.0 mm
- net /CODEC/LINEOUT_L: track 0.00 -> 16.3 mm, vias 0 -> 1
- net /CODEC/I2C_SDA: track 0.00 -> 14.8 mm
- net /CODEC/I2S_DIN: track 0.00 -> 11.7 mm
- net /CODEC/SYS_MCLK: track 0.00 -> 10.1 mm
- net /CODEC/I2S_DOUT: track 0.00 -> 8.51 mm
- net /CODEC/I2S_LRCLK: track 0.00 -> 7.60 mm
- net /CODEC/I2S_SCLK: track 0.00 -> 5.81 mm
- net /STM32/SYS_MCLK: track 0.00 -> 2.67 mm
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- added copper zone on F.Cu, net GND

Commit message: Started routing
Parts:
- C202, C203: footprint Capacitor_SMD:C_0603_1608Metric -> Capacitor_SMD:C_0402_1005Metric
- R204: footprint Resistor_SMD:R_0603_1608Metric -> Resistor_SMD:R_0402_1005Metric
- moved C203 43.3 mm to (62.2, 61.6), turned to 180 degrees
- moved TP502 41.1 mm to (91.0, 48.0)
- moved R202 40.9 mm to (68.5, 50.5), turned to 0 degrees
- moved R204 40.4 mm to (70.6, 53.9)
- moved Y201 39.5 mm to (62.2, 58.8)
- moved R503 39.5 mm to (38.5, 50.0), turned to 180 degrees
- moved SW201 39.4 mm to (64.0, 66.0)
- moved R203 39.3 mm to (66.0, 58.8)
- moved R502 39.0 mm to (91.0, 54.5), turned to -90 degrees
- moved C205 39.0 mm to (68.3, 55.3)
- moved C201 38.7 mm to (66.6, 60.2)
- moved U201 38.6 mm to (73.0, 60.0)
- moved C204 38.3 mm to (79.0, 67.4)
- moved R201 38.2 mm to (68.5, 48.5), turned to 0 degrees
- moved C206 38.2 mm to (77.7, 64.7)
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Routing:
- net /STM32/I2C_SCL: track 2.67 -> 44.5 mm, vias 0 -> 2
- net /STM32/I2S_DIN: track 2.67 -> 40.3 mm, vias 0 -> 2
- net /CODEC/MIC: track 69.6 -> 34.1 mm, vias 0 -> 1
- net GND: track 0.00 -> 35.3 mm, vias 0 -> 43
- net /STM32/I2C_SDA: track 2.67 -> 37.9 mm, vias 0 -> 2
- net /STM32/I2S_DOUT: track 2.67 -> 34.3 mm
- net /STM32/VCP_TX: track 0.00 -> 18.7 mm, vias 0 -> 2
- net /STM32/nRST: track 0.00 -> 17.3 mm, vias 0 -> 2
- net /STM32/VCP_RX: track 0.00 -> 16.8 mm
- net /CODEC/LINEOUT_R: track 26.7 -> 42.6 mm
- net /STM32/SYS_MCLK: track 2.67 -> 15.7 mm
- net /STM32/I2S_SCLK: track 18.1 -> 30.3 mm, vias 0 -> 2
- net /STM32/OSC_IN: track 0.00 -> 8.13 mm
- net /STM32/SWO: track 0.00 -> 7.50 mm
- net /STM32/XTAL_OUT: track 0.00 -> 6.85 mm
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- added copper zone on In1.Cu, net GND
Other:
- board size 68 x 68 mm -> 88 x 38 mm
- copper layers 2 -> 4
- board text added: "+"

Commit message: routing
Parts:
- moved D201 26.9 mm to (83.0, 68.5)
- moved D202 26.9 mm to (83.0, 70.5)
- moved R201 26.9 mm to (86.5, 68.5)
- moved R202 26.9 mm to (86.5, 70.5)
- moved C204 0.90 mm to (79.0, 66.5)
- moved C302 0.60 mm to (52.8, 64.2)
Connections:
- U201 pad 10: unconnected-(U201-PA5-Pad10) -> /STM32/LED1
- U201 pad 5: /STM32/LED1 -> unconnected-(U201-PA0-Pad5)
- U201 pad 6: /STM32/LED2 -> unconnected-(U201-PA1-Pad6)
- U201 pad 9: unconnected-(U201-PA4-Pad9) -> /STM32/LED2
Routing:
- net +5V: track 0.00 -> 27.5 mm, vias 0 -> 9
- net /STM32/LED2: track 0.00 -> 17.2 mm
- net /STM32/USB_D+: track 0.00 -> 16.2 mm
- net /STM32/USB_D-: track 0.00 -> 16.0 mm
- net +3V3: track 3.70 -> 19.4 mm, vias 0 -> 9
- net /POWER/VBUS: track 1.52 -> 16.9 mm, vias 1 -> 4
- net /STM32/LED1: track 0.00 -> 15.1 mm
- net +3.3VA: track 1.44 -> 14.0 mm, vias 0 -> 5
- net /STM32/nRST: track 17.3 -> 24.2 mm, vias 2 -> 4
- net +1V8: track 3.70 -> 10.1 mm, vias 0 -> 3
- net /USB/CC1: track 0.00 -> 4.09 mm
- net /USB/CC2: track 0.00 -> 3.94 mm
- net /POWER/FUSE: track 0.00 -> 3.14 mm
- net /POWER/LED33_MID: track 0.00 -> 1.89 mm
- net /POWER/LED33A_MID: track 0.00 -> 1.89 mm
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- added copper zone on In2.Cu, net +1V8
- added copper zone on In2.Cu, net +3.3VA
- added copper zone on In2.Cu, net +3V3
- added copper zone on In2.Cu, net +5V
- added copper zone on B.Cu, net GND

Commit message: finished routing
Routing:
- net GND: vias 45 -> 143
Other:
- board text added: "+1V8"
- board text added: "+3.3VA"
- board text added: "+3V3"
- board text added: "DIN"
- board text added: "DOUT"
- board text added: "LINEIN_L"
- board text added: "LINEIN_R"
- board text added: "LINEOUT_L"
- board text added: "LINEOUT_R"
- board text added: "LR"
- board text added: "MCLK"
- board text added: "MIC"
- board text added: "RESET"
- board text added: "SCL"
- board text added: "SCLK"
- board text added: "SDA"
- board text added: "Test SGTL5000 Laurent Fiack 11/05/2023 rev 1.0"
